Commit message: Fixed collision, added key press robot control

File: robusser_robot.urdf (robot description, URDF)
Before this commit: robot mmp_panda, 13 links, 12 joints
Links:
- link base_link: geometry collision box size=0.44 0.44 0.3; visual mesh filename=../../../model/mmp_panda/meshes/panda_BaseCombo.obj
- link link1: geometry collision mesh filename=../../../model/panda/meshes/collision/link1.obj; visual mesh filename=../../../model/panda/meshes/visual/link1.obj
- link link2: geometry collision mesh filename=../../../model/panda/meshes/collision/link2.obj; visual mesh filename=../../../model/panda/meshes/visual/link2.obj
- link link3: geometry collision mesh filename=../../../model/panda/meshes/collision/link3.obj; visual mesh filename=../../../model/panda/meshes/visual/link3.obj
- link link4: geometry collision mesh filename=../../../model/panda/meshes/collision/link4.obj; visual mesh filename=../../../model/panda/meshes/visual/link4.obj
- link link5: geometry collision mesh filename=../../../model/panda/meshes/collision/link5.obj; visual mesh filename=../../../model/panda/meshes/visual/link5.obj
- link link6: geometry collision mesh filename=../../../model/panda/meshes/collision/link6.obj; visual mesh filename=../../../model/panda/meshes/visual/link6.obj
- link link7: geometry collision mesh filename=../../../model/panda/meshes/collision/hand.obj; collision mesh filename=../../../model/panda/meshes/collision/link7.obj

Commit message: Improved controller organization and added dishwasher bot

File: robusser_robot.urdf (robot description, URDF)
Before this commit: robot mmp_panda, 13 links, 12 joints
Links:
- link link1: geometry visual mesh filename=../../../model/panda/meshes/visual/link1.obj
- link link2: geometry visual mesh filename=../../../model/panda/meshes/visual/link2.obj
- link link3: geometry visual mesh filename=../../../model/panda/meshes/visual/link3.obj
- link link4: geometry visual mesh filename=../../../model/panda/meshes/visual/link4.obj
- link link5: geometry visual mesh filename=../../../model/panda/meshes/visual/link5.obj
- link link6: geometry visual mesh filename=../../../model/panda/meshes/visual/link6.obj
- link link7: geometry visual mesh filename=../../../model/panda/meshes/visual/hand.obj; visual mesh filename=../../../model/panda/meshes/visual/link7.obj

Commit message: add controls

File: robusser_robot.urdf (robot description, URDF)
Before this commit: robot mmp_panda, 13 links, 12 joints
Links:
- link link7: geometry collision mesh filename=../../../model/panda/meshes/collision/link7.obj; visual mesh filename=../../../model/panda/meshes/visual/hand.obj

Commit message: update

File: robusser_robot.urdf (robot description, URDF)
Before this commit: robot mmp_panda, 13 links, 12 joints
Links:
- link leftfinger: geometry collision box size=.01 .01 .11; visual box size=.01 .01 .11
- link link7: geometry collision mesh filename=../../../model/panda/meshes/collision/hand.obj; collision mesh filename=../../../model/panda/meshes/collision/link7.obj
- link rightfinger: geometry collision box size=.01 .01 .11; visual box size=.01 .01 .11
